File: EIT_3/Schaltungstechnik/Labor/Labor1/waage_ina155_ad8041/waage_ina155_ad8041.kicad_pcb (KiCad board)
At the start: 2 copper layers, 76.2 x 44.4 mm, 26 parts, among them J1 Conn_01x03_Pin, J2 Conn_01x04_Pin

Commit message: Auto-Update PC-zuhause 2025-12-14 14:16
Routing:
- net GND: track 147.0 -> 138.1 mm
- net Net-(U1-Ref): track 56.5 -> 55.9 mm
Other:
- outline, holes or cut-outs redrawn
Changed lines of the file:
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@@
 	)
 	(gr_circle
-		(center 116.84 91.690665)
-		(end 118.11 90.420665)
+		(center 131.145898 96)
+		(end 132.645898 99)
 		(stroke
 			(width 0.05)
@@
 	)
 	(gr_circle
-		(center 186.163949 123.19)
-		(end 187.433949 121.92)
+		(center 185 121.5)
+		(end 186.5 124.5)
 		(stroke
 			(width 0.05)
@@
 	)
 	(gr_circle
-		(center 118.11 123.440665)
-		(end 116.313949 122.170665)
-		(stroke
-			(width 0.05)
-			(type default)
-		)
-		(fill no)
-		(layer "Edge.Cuts")
-	)
-	(gr_circle
-		(center 187.96 91.44)
-		(end 189.23 90.17)
+		(center 131.145898 121.5)
+		(end 132.645898 124.5)
 		(stroke
 			(width 0.05)
@@
 	)
 	(segment
-		(start 173.985121 102.875037)
-		(end 173.9868 102.876716)
-		(width 0.5)
-		(layer "F.Cu")
-		(net 2)
-	)
-	(segment
 		(start 136.983128 115.534919)
 		(end 137.146527 115.37152)
@@
 	)
 	(segment
-		(start 182.8768 97.796716)
-		(end 174.01745 97.796716)
-		(width 0.75)
-		(layer "F.Cu")
-		(net 2)
-	)
-	(segment
 		(start 153.6668 103.575521)
 		(end 152.792162 103.575521)
@@
 	)
 	(segment
-		(start 160.950746 101.163251)
-		(end 160.950746 101.168688)
-		(width 0.5)
-		(layer "F.Cu")
-		(net 2)
-	)
-	(segment
 		(start 163.8268 128.276716)
 		(end 176.53 128.276716)
@@
 	)
 	(segment
-		(start 163.810851 122.561023)
-		(end 163.780048 122.53022)
-		(width 0.75)
-		(layer "F.Cu")
-		(net 2)
-	)
-	(segment
 		(start 137.1568 115.37152)
 		(end 137.689202 114.839118)
@@
 	)
 	(segment
-		(start 119.6308 109.226716)
-		(end 119.6054 109.201316)
-		(width 0.5)
-		(layer "F.Cu")
-		(net 4)
-	)
-	(segment
 		(start 121.8914 109.201316)
 		(end 121.9168 109.226716)
@@
 	)
 	(segment
-		(start 140.126814 111.131506)
-		(end 140.204913 111.053407)
-		(width 0.5)
-		(layer "F.Cu")
-		(net 5)
-	)
-	(segment
 		(start 130.8068 113.036716)
 		(end 120.9008 113.036716)
@@
 		(width 0.5)
 		(layer "F.Cu")
-		(net 9)
-	)
-	(segment
-		(start 168.693105 97.300892)
-		(end 168.132624 97.300892)
-		(width 0.5)
-		(layer "F.Cu")

Commit message: Auto-Update PC-zuhause 2025-12-14 14:31
Other:
- board text added: "3V3"
Changed lines of the file:
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@@
 			(outputformat 1)
 			(mirror no)
-			(drillshape 1)
+			(drillshape 0)
 			(scaleselection 1)
 			(outputdirectory "")
@@
 	)
 	(gr_text "GND"
+		(at 121.449677 115.091643 0)
+		(layer "F.SilkS")
+		(effects
+			(font
+				(size 1 1)
+				(thickness 0.1)
+			)
+			(justify left bottom)
+		)
+	)
+	(gr_text "GND"
 		(at 118.688684 127.900963 0)
 		(layer "F.SilkS")
@@
 		)
 	)
+	(gr_text "3V3"
+		(at 180.992908 108.63224 0)
+		(layer "F.SilkS")
+		(effects
+			(font
+				(size 1 1)
+				(thickness 0.1)
+			)
+			(justify left bottom)
+		)
+	)
 	(gr_text "GND"
 		(at 179.408266 127.753603 0)
@@
 		)
 	)
+	(gr_text "3V3"
+		(at 121.349031 107.241294 0)
+		(layer "F.SilkS")
+		(effects
+			(font
+				(size 1 1)
+				(thickness 0.1)
+			)
+			(justify left bottom)
+		)
+	)
 	(gr_text "AD8041"
 		(at 165.216452 125.126695 0)
@@
 				(thickness 0.1)
 			)
+			(justify left bottom)
+		)
+	)
+	(gr_text "GND"
+		(at 180.841939 113.731612 0)
+		(layer "F.SilkS")
+		(effects
+			(font
+				(size 1 1)
+				(thickness 0.1)
+			)
